File: PCB Files/Rev 1/Order.brd (EAGLE design)
At the start: 115 x 111 mm, 67 parts, among them IC2 ATMEGA328P, J1 USB4085-GF-A_REVA, SW1 EC12E_SW, X1 49S/18PF

Commit message: new LED placement...
I basicly redrew every trace
Parts:
- added LED5: WS2812B, SparkFun-LED:WS2812B
- moved LED1 42.5 mm to (19.5, 19.5)
- moved LED4 42.5 mm to (76.5, 19.5)
- moved LED2 19.0 mm to (38.5, 19.5)
- moved LED3 19.0 mm to (57.5, 19.5)
- moved SW1 4.00 mm to (86.0, 10.0)
Connections:
- new net N$5: LED4.2, LED5.4
- net 5V: now also LED5.1
- net GND: now also LED5.3
Routing:
- net GND: track 315.3 -> 277.5 mm
- net 5V: track 207.3 -> 233.5 mm, vias 2 -> 0
- net RGB_DATA: track 79.4 -> 95.1 mm, vias 2 -> 1
- net N$5: track 0.00 -> 15.2 mm
- net LED-: track 403.5 -> 392.9 mm
- net N$46: track 25.4 -> 15.2 mm, vias 2 -> 0
- net ROW2: track 95.6 -> 86.0 mm
- net LED+: track 396.4 -> 401.9 mm
- net ROW3: track 93.2 -> 90.3 mm
- net N$60: track 72.6 -> 75.5 mm
- net N$75: track 90.7 -> 93.4 mm
- net N$77: track 90.7 -> 93.4 mm
- net N$62: track 72.7 -> 75.4 mm
- net N$41: track 17.9 -> 15.2 mm, vias 2 -> 0
- net COLUMN2: track 72.7 -> 70.3 mm
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